File: Power Design/PowerDelivery/PowerDelivery.kicad_sch (KiCad schematic)
At the start: 29 parts, among them J1 Conn_01x06_Pin, J2 Conn_01x24_Socket, J3 Screw_Terminal_01x08, Q1 Q_NPN_CBE, U1 Opamp_Dual, U2 Opamp_Dual, U3 2EDN8524FXTMA1, U4 IPP016N06NF2SAKMA1, U5 Opamp_Dual

Commit message: initial commit
Parts:
- added H1, H2, H3, H4: MountingHole_Pad, MountingHole:MountingHole_3.2mm_M3_ISO7380_Pad, symbol Mechanical:MountingHole_Pad
- added R17, R18: 1K, Resistor_SMD:R_0805_2012Metric_Pad1.20x1.40mm_HandSolder, symbol Device:R
- J1: footprint Connector_Molex:Molex_Mini-Fit_Jr_5566-06A_2x03_P4.20mm_Vertical -> Connector_PinHeader_2.54mm:PinHeader_1x06_P2.54mm_Vertical
Connections:
- net GND: now also H1.1, H2.1, H3.1, H4.1
- net current_sense_out: now also R17.2; no longer U2.6 (-), U2.7
- net voltage_sense_out: now also R18.2; no longer U1.6 (-), U1.7
- new net: R17.1, U2.7
- new net: R18.1, U1.7

Commit message: initial commit
Parts:
- added J4: 8 Pin EPS, Connector_Molex:Molex_Mini-Fit_Jr_5566-08A_2x04_P4.20mm_Vertical, symbol Connector_Generic:Conn_02x04_Top_Bottom
- added J5: PS-ON, Connector_PinHeader_2.54mm:PinHeader_1x02_P2.54mm_Vertical, symbol Connector_Generic:Conn_01x02
- J2: value Conn_01x24_Socket -> 24 Pin ATX
Connections:
- net +12V: now also J4.5 (Pin_5), J4.6 (Pin_6), J4.7 (Pin_7), J4.8 (Pin_8)
- net GND: now also J4.1 (Pin_1), J4.2 (Pin_2), J4.3 (Pin_3), J4.4 (Pin_4), J5.1 (Pin_1)
- net at J2.16 (Pin_16): now also J5.2 (Pin_2)
Other:
- note added: "PSU Connectors"
- note removed: "PSU Connector"

Commit message: Create power delivery V2
Connections:
- net +3.3V: now also J1.2 (Pin_2); no longer J1.6 (Pin_6), J2.12 (Pin_12)
- net GND: now also C2.1, J1.1 (Pin_1); no longer C2.2, J1.5 (Pin_5)
- net current_sense_out: now also J1.5 (Pin_5); no longer J1.1 (Pin_1)
- net voltage_sense_out: now also J1.6 (Pin_6); no longer J1.2 (Pin_2)
- net at R17.1, U2.7: now also U2.6 (-)
- net at Q1.2 (B), R15.2: now also C2.2; no longer C2.1
- net at R18.1, U1.7: now also U1.6 (-)
Other:
- moved on the sheet: C2
Changed lines of the file:
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@@
 	)
 	(junction
+		(at 133.35 43.18)
+		(diameter 0)
+		(color 0 0 0 0)
+	)
+	(junction
 		(at 252.73 134.62)
 		(diameter 0)
@@
 		(color 0 0 0 0)
 	)
+	(junction
+		(at 35.56 41.91)
+		(diameter 0)
+		(color 0 0 0 0)
+	)
 	(wire
 		(pts
@@
 	(wire
 		(pts
+			(xy 35.56 41.91) (xy 35.56 49.53)
+		)
+		(stroke
+			(width 0)
+			(type default)
+		)
+	)
+	(wire
+		(pts
 			(xy 170.18 45.72) (xy 170.18 43.18)
 		)
@@
 	(wire
 		(pts
+			(xy 133.35 43.18) (xy 133.35 50.8)
+		)
+		(stroke
+			(width 0)
+			(type default)
+		)
+	)
+	(wire
+		(pts
 			(xy 50.8 39.37) (xy 53.34 39.37)
 		)
@@
 	(global_label "voltage_sense_out"
 		(shape input)
-		(at 248.92 35.56 0)
+		(at 248.92 45.72 0)
 		(fields_autoplaced yes)
 		(effects
@@
 		)
 		(property "Intersheetrefs" "${INTERSHEET_REFS}"
-			(at 269.0612 35.56 0)
+			(at 269.0612 45.72 0)
 			(effects
 				(font
@@
 	(global_label "current_sense_out"
 		(shape input)
-		(at 248.92 33.02 0)
+		(at 248.92 43.18 0)
 		(fields_autoplaced yes)
 		(effects
@@
 		)
 		(property "Intersheetrefs" "${INTERSHEET_REFS}"
-			(at 268.9404 33.02 0)
+			(at 268.9404 43.18 0)
 			(effects
 				(font
@@
 	(symbol
 		(lib_id "Device:C")
-		(at 148.59 147.32 0)
+		(at 148.59 147.32 180)
 		(unit 1)
 		(exclude_from_sim no)
@@
 		(fields_autoplaced yes)
 		(property "Reference" "C2"
-			(at 152.4 146.685 0)
+			(at 152.4 146.0499 0)
 			(effects
 				(font
 					(size 1.27 1.27)
 				)
-				(justify left)
+				(justify right)
 			)
 		)
 		(property "Value" "1n"
-			(at 152.4 149.225 0)
+			(at 152.4 148.5899 0)
 			(effects
 				(font
 					(size 1.27 1.27)
 				)
-				(justify left)
+				(justify right)
 			)
 		)
 		(property "Footprint" "Capacitor_SMD:C_0805_2012Metric_Pad1.18x1.45mm_HandSolder"
-			(at 149.5552 151.13 0)
+			(at 147.6248 143.51 0)
 			(effects
 				(font
@@
 	(symbol
 		(lib_id "power:GND")
-		(at 248.92 43.18 90)
+		(at 248.92 33.02 90)
 		(unit 1)
 		(exclude_from_sim no)
@@
 		(fields_autoplaced yes)
 		(property "Reference" "#PWR08"
-			(at 255.27 43.18 0)
+			(at 255.27 33.02 0)
 			(effects
 				(font
@@
 		)
 		(property "Value" "GND"
-			(at 252.73 43.815 90)
+			(at 252.73 33.655 90)
 			(effects
 				(font
@@
 		)
 		(property "Footprint" ""
-			(at 248.92 43.18 0)
+			(at 248.92 33.02 0)
 			(effects
 				(font
@@
 		)
 		(property "Datasheet" ""
-			(at 248.92 43.18 0)
+			(at 248.92 33.02 0)
 			(effects
 				(font
@@
 		)
 		(property "Description" ""
-			(at 248.92 43.18 0)
+			(at 248.92 33.02 0)
 			(effects
 				(font
@@
 	(symbol
 		(lib_id "power:+3.3V")
-		(at 248.92 45.72 270)
+		(at 248.92 35.56 270)
 		(unit 1)
 		(exclude_from_sim no)
@@
 		(fields_autoplaced yes)
 		(property "Reference" "#PWR09"
-			(at 245.11 45.72 0)
+			(at 245.11 35.56 0)
 			(effects
 				(font
@@
 		)
 		(property "Value" "+3.3V"
-			(at 252.73 46.355 90)
+			(at 252.73 36.195 90)
 			(effects
 				(font
@@
 		)
 		(property "Footprint" ""
-			(at 248.92 45.72 0)
+			(at 248.92 35.56 0)
 			(effects
 				(font
@@
 		)
 		(property "Datasheet" ""
-			(at 248.92 45.72 0)
+			(at 248.92 35.56 0)
 			(effects
 				(font
@@
 		)
 		(property "Description" ""
-			(at 248.92 45.72 0)
+			(at 248.92 35.56 0)
 			(effects
 				(font
@@
 					(unit 1)
 				)
-			)
-		)
-	)
-	(symbol
-		(lib_id "power:+3.3V")
-		(at 251.46 92.71 90)
-		(unit 1)
-		(exclude_from_sim no)
-		(in_bom yes)
-		(on_board yes)
-		(dnp no)
-		(fields_autoplaced yes)
-		(property "Reference" "#PWR021"
-			(at 255.27 92.71 0)
-			(effects
-				(font
-					(size 1.27 1.27)
-				)
-				(hide yes)
-			)
-		)
-		(property "Value" "+3.3V"
-			(at 247.65 93.345 90)
-			(effects
-				(font
-					(size 1.27 1.27)
-				)
-				(justify left)
-			)
-		)
-		(property "Footprint" ""
-			(at 251.46 92.71 0)
-			(effects
-				(font
-					(size 1.27 1.27)
-				)
-				(hide yes)
-			)
-		)
-		(property "Datasheet" ""
-			(at 251.46 92.71 0)
-			(effects
-				(font
-					(size 1.27 1.27)
-				)
-				(hide yes)
-			)
-		)
-		(property "Description" ""
-			(at 251.46 92.71 0)
-			(effects
-				(font
-					(size 1.27 1.27)
-				)
-				(hide yes)
-			)
-		)
-		(pin "1"
-		)
-		(instances
-			(project "PowerDelivery"
-				(path "/40c9a0c2-e09d-483c-9187-ad4dcc209d53"
-					(reference "#PWR021")
-					(unit 1)
-				)

Commit message: Change implemented
Parts:
- removed J3: Screw_Terminal_01x08, Home_Made:YK4410403000G, symbol Connector:Screw_Terminal_01x08
- added C3, C4, C5, C6, C7: 200n, Capacitor_THT:C_Disc_D3.8mm_W2.6mm_P2.50mm, symbol Device:C
- added D2: LED, LED_THT:LED_D5.0mm, symbol Device:LED
- added J3, J6, J7, J8: Screw_Terminal_01x02, TerminalBlock:TerminalBlock_bornier-2_P5.08mm, symbol Connector:Screw_Terminal_01x02
- C1: value 100n -> 20n; footprint Capacitor_SMD:C_0805_2012Metric_Pad1.18x1.45mm_HandSolder -> Capacitor_THT:C_Disc_D3.8mm_W2.6mm_P2.50mm
- C2: value 1n -> 200n; footprint Capacitor_SMD:C_0805_2012Metric_Pad1.18x1.45mm_HandSolder -> Capacitor_THT:C_Disc_D3.8mm_W2.6mm_P2.50mm
- D1: footprint Diode_SMD:D_0805_2012Metric_Pad1.15x1.40mm_HandSolder -> Diode_THT:D_DO-41_SOD81_P7.62mm_Horizontal
- Q1: value Q_NPN_CBE -> PN2222ATA; footprint Package_TO_SOT_SMD:SOT-23 -> Package_TO_SOT_THT:TO-92_Wide
- R1, R8: value 100K -> 1K; footprint Resistor_SMD:R_0805_2012Metric_Pad1.20x1.40mm_HandSolder -> Resistor_THT:R_Axial_DIN0207_L6.3mm_D2.5mm_P7.62mm_Horizontal
- R10, R11, R12, R13, R14, R17, R18, R4, R7: footprint Resistor_SMD:R_0805_2012Metric_Pad1.20x1.40mm_HandSolder -> Resistor_THT:R_Axial_DIN0207_L6.3mm_D2.5mm_P7.62mm_Horizontal
- R15: value 1K -> 4.7K; footprint Resistor_SMD:R_0805_2012Metric_Pad1.20x1.40mm_HandSolder -> Resistor_THT:R_Axial_DIN0207_L6.3mm_D2.5mm_P7.62mm_Horizontal
- R16: value 22 -> 4.7K; footprint Resistor_SMD:R_0805_2012Metric_Pad1.20x1.40mm_HandSolder -> Resistor_THT:R_Axial_DIN0207_L6.3mm_D2.5mm_P7.62mm_Horizontal
- R2, R9: value 100K -> 4K; footprint Resistor_SMD:R_0805_2012Metric_Pad1.20x1.40mm_HandSolder -> Resistor_THT:R_Axial_DIN0207_L6.3mm_D2.5mm_P7.62mm_Horizontal
- R3, R5: value 100K -> 10K; footprint Resistor_SMD:R_0805_2012Metric_Pad1.20x1.40mm_HandSolder -> Resistor_THT:R_Axial_DIN0207_L6.3mm_D2.5mm_P7.62mm_Horizontal
- R6: footprint Home_Made:SR52L500FE66 -> Resistor_THT:R_Axial_DIN0617_L17.0mm_D6.0mm_P20.32mm_Horizontal
- RV1: footprint Potentiometer_SMD:Potentiometer_Bourns_3224W_Vertical -> Potentiometer_THT:Potentiometer_Bourns_3296W_Vertical
- U1, U2, U5: value Opamp_Dual -> LM258AP; footprint Package_SO:SOIC-8_3.9x4.9mm_P1.27mm -> Package_DIP:DIP-8_W7.62mm
- U3: value 2EDN8524FXTMA1 -> UCC27524P; footprint Home_Made:Infineon_PG-DSO-8-60 -> Package_DIP:DIP-8_W7.62mm
Connections:
- net +12V: now also C2.1, R16.2, C5.1, C7.1, J7.1 (Pin_1), J7.2 (Pin_2), J8.1 (Pin_1), J8.2 (Pin_2)
- net -12V: now also C3.1, C4.1, C6.1
- net GND: now also C2.2, C3.2, C4.2, C5.2, C6.2, C7.2, D2.1 (K); no longer C2.1
- net load: now also J3.1 (Pin_1), J3.2 (Pin_2), J6.1 (Pin_1), J6.2 (Pin_2)
- net at Q1.2 (B), R15.2: no longer C2.2
- net at C1.1, U3.1 (ENA), U3.8 (ENB): now also Q1.1 (C); no longer R16.2
- net at R16.1: now also D2.2 (A); no longer Q1.1 (C)
Other:
- moved on the sheet: U1C, U2C
