File: Power Design/PowerDelivery/PowerDelivery.kicad_pcb (KiCad board)
At the start: 2 copper layers, 85 x 85 mm, 47 parts, among them J1 Conn_01x06_Pin, J2 24 Pin ATX, J3 Screw_Terminal_01x02, J4 8 Pin EPS, J5 PS-ON, J6 Screw_Terminal_01x02, J7 Screw_Terminal_01x02, J8 Screw_Terminal_01x02, Q1 PN2222ATA, U1 LM258AP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

Commit message: Made changes from v3
Parts:
- moved J5 17.9 mm to (128.5, 78.2), turned to 180 degrees
- moved C1 9.51 mm to (180.5, 113.8)
- moved C2 9.51 mm to (173.8, 126.0)
- moved C3 9.51 mm to (162.8, 138.0)
- moved C4 9.51 mm to (152.2, 81.5)
- moved C5 9.51 mm to (164.0, 92.2)
- moved C6 9.51 mm to (152.8, 101.0)
- moved C7 9.51 mm to (150.8, 116.0)
- moved D1 9.51 mm to (175.5, 69.7)
- moved D2 9.51 mm to (167.8, 120.5)
- moved Q1 9.51 mm to (175.8, 115.0)
- moved R1 9.51 mm to (150.7, 135.5)
- moved R10 9.51 mm to (172.0, 77.2)
- moved R11 9.51 mm to (179.5, 69.7)
- moved R12 9.51 mm to (173.7, 90.0)
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Routing:
- net load: track 83.8 -> 97.1 mm
- net +12V: track 132.3 -> 119.7 mm
- net Net-(D1-K): track 35.4 -> 23.2 mm, vias 0 -> 9
- net -12V: track 101.6 -> 89.9 mm
- net fault_signal: track 27.5 -> 16.2 mm
- net voltage_sense_out: track 40.7 -> 30.6 mm
- net mc_trigger: track 24.4 -> 14.7 mm
- net current_sense_out: track 29.1 -> 19.8 mm
- net Net-(J2-Pin_16): track 14.9 -> 7.35 mm
- net Net-(D1-A): track 44.1 -> 39.5 mm
- net Net-(U3-OUTA): track 31.9 -> 29.9 mm
- net +3.3V: track 76.9 -> 75.2 mm
- net Net-(Q1-C): track 23.0 -> 23.7 mm
- net Net-(U4-GATE): track 34.6 -> 34.0 mm
- net GND: vias 9 -> 0
- added copper zone on B.Cu, net Net-(D1-K)
- added copper zone on F.Cu, net Net-(D1-K)
Other:
- board text added: "3"
- board text added: "Octoforge power delivery v4"
- board text removed: "Octoforge power delivery v3"
